Commit message: feat: Phase 2C — runnable Gazebo simulation
New EJS templates:
- sim/gazebo/world.sdf.ejs — full Gazebo world with robot model
  - Differential drive plugin (libgazebo_ros_diff_drive)
  - LiDAR sensor with ray plugin (libgazebo_ros_ray_sensor)
  - IMU sensor with noise model (libgazebo_ros_imu_sensor)
  - Wheel joints with dynamics (damping, friction)
  - Proper physics config (ODE, 1000 Hz)
  - Auto-detects sensor types from hardware description
- ros2/launch/sim.launch.py.ejs — simulation launch
  - Gazebo launch + robot_state_publisher + spawner
  - ros2_control with diff_drive_controller + joint_state_broadcaster
  - use_sim_time for all nodes

Updated generators:
- gazebo.ts — now uses EJS template instead of inline string,
  generates proper world with all sensor plugins,
  accepts KnowledgeContext for motor/sensor resolution,
  writes docker/entrypoint.sh with exec permissions
- ros2-driver.ts — generates sim.launch.py when --sim flag set,
  passes robotName/rosNs/pkgName to templates
- urdf.ts — accepts optional KnowledgeContext parameter
- index.ts — passes kb to generateGazebo and generateUrdf

Docker Compose:
- Uses osrf/ros:humble-desktop-full (official ROS 2 + Gazebo image)
- NVIDIA GPU passthrough
- Volume mounts for sim/, urdf/, ros2_ws/
- Entrypoint script for source setup

Output:
- diff-drive demo now generates 13 files (was 11)
- New: sim/gazebo/*.sdf (30 plugin/sensor/joint elements)
- New: sim.launch.py (Gazebo + controllers + spawning)
- New: docker/entrypoint.sh

19 tests all passing, no regressions

File: examples/diff-drive-inspector/generated/urdf/巡检机器人-c3.urdf.xacro (robot description, xacro)
@@ -2,7 +2,7 @@
 <!--
 Robot URDF/XACRO — Auto-generated by Hermod
-@ai-context: This URDF describes the full kinematic tree of the robot.
+@ai-context: This URDF describes the full kinematic tree of 巡检机器人-C3.
+Type: diff_drive.
 Link origins and joint axes are derived from robot.hardware.yaml.
-Sensor mount positions are included as static transforms.
 Mass/inertia values are placeholders — replace with CAD-derived values.
 @ai-extend: Add custom links, gazebo plugins, or transmission blocks below.
@@ -10,32 +10,36 @@
 <robot xmlns:xacro="http://www.ros.org/wiki/xacro" name="______C3">
 <!-- ── Materials ── -->
-<material name="chassis_grey">
-<color rgba="0.4 0.4 0.4 1"/>
+<material name="base_grey">
+<color rgba="0.3 0.3 0.3 1"/>
 </material>
-<material name="wheel_black">
-<color rgba="0.1 0.1 0.1 1"/>
+<material name="link_grey">
+<color rgba="0.5 0.5 0.5 1"/>
 </material>
 <material name="sensor_blue">
 <color rgba="0.2 0.4 0.8 1"/>
 </material>
-<!-- ── Base Link ── -->
+<!-- ═══════════════════════════════════════ -->
+<!-- Base Link                               -->
+<!-- ═══════════════════════════════════════ -->
 <link name="base_link">
 <inertial>
-<mass value="1.0"/>  <!-- TODO: replace with actual mass -->
-<inertia ixx="0.1" ixy="0" ixz="0" iyy="0.1" iyz="0" izz="0.1"/>
+<mass value="3.0"/>
+<inertia ixx="0.2" ixy="0" ixz="0" iyy="0.2" iyz="0" izz="0.2"/>
 </inertial>
 <visual>
 <geometry>
-<box size="0.3 0.2 0.15"/>
+<box size="0.4 0.25 0.15"/>
 </geometry>
-<material name="chassis_grey"/>
+<material name="base_grey"/>
 </visual>
 <collision>
 <geometry>
-<box size="0.3 0.2 0.15"/>
+<box size="0.4 0.25 0.15"/>
 </geometry>
 </collision>
 </link>
-<!-- ── Wheels ── -->
+<!-- ═══════════════════════════════════════ -->
+<!-- Mobile Base (Wheels)                    -->
+<!-- ═══════════════════════════════════════ -->
 <!-- Active: left_front_wheel (Motor: dji-m3508) -->
 <link name="left_front_wheel">
@@ -45,8 +49,5 @@
 </inertial>
 <visual>
-<geometry>
-<cylinder radius="0.06" length="0.03"/>
-</geometry>
-<material name="wheel_black"/>
+<geometry><cylinder radius="0.06" length="0.03"/></geometry>
 </visual>
 </link>
@@ -64,8 +65,5 @@
 </inertial>
 <visual>
-<geometry>
-<cylinder radius="0.06" length="0.03"/>
-</geometry>
-<material name="wheel_black"/>
+<geometry><cylinder radius="0.06" length="0.03"/></geometry>
 </visual>
 </link>
@@ -83,8 +81,5 @@
 </inertial>
 <visual>
-<geometry>
-<cylinder radius="0.06" length="0.03"/>
-</geometry>
-<material name="wheel_black"/>
+<geometry><cylinder radius="0.06" length="0.03"/></geometry>
 </visual>
 </link>
@@ -102,8 +97,5 @@
 </inertial>
 <visual>
-<geometry>
-<cylinder radius="0.06" length="0.03"/>
-</geometry>
-<material name="wheel_black"/>
+<geometry><cylinder radius="0.06" length="0.03"/></geometry>
 </visual>
 </link>
@@ -121,7 +113,5 @@
 </inertial>
 <visual>
-<geometry>
-<box size="0.03 0.03 0.03"/>
-</geometry>
+<geometry><box size="0.03 0.03 0.03"/></geometry>
 <material name="sensor_blue"/>
 </visual>
@@ -139,7 +129,5 @@
 </inertial>
 <visual>
-<geometry>
-<box size="0.03 0.03 0.03"/>
-</geometry>
+<geometry><box size="0.03 0.03 0.03"/></geometry>
 <material name="sensor_blue"/>
 </visual>
